File: ev-microcontroller.kicad_sch (KiCad schematic)
At the start: 0 parts

Commit message: First major revision
Other:
- added sheet Connectors (conenctors.kicad_sch)
- added sheet MCU (mcu.kicad_sch)
- added sheet Memory (memory.kicad_sch)
- added sheet Peripherals (peripherals.kicad_sch)
- added sheet Power (power.kicad_sch)
- note added: "Description ----------- The EV Microcontroller is a small, portable, self-contained processing unit that is capable of reading in sensor data and outputing that data to a CAN bus. It is meant to be a robust alternative to a similar unit made of an arduino and compatable shields."
- note added: "EV Microcontroller"
- note added: "Features -------- Low power, shock resistant CAN connectivity 5 12-bit analog pins 10 digital pins Micropython support RP2040 microprocessor Onboard power distribution (3V3, 5V, 12V) USB-C flash/debug/power/data port MicroSD CAN backup M2 grounded mounting holes Board thermistor 9 axis gyroscope Compact (30mm x 40mm) Electrical protections (overcurrent, undervoltage, etc.)"
- note added: "Page | Description -------------- 01 Index Page 02 MCU 03 Power 04 Memory 05 Peripherals 06 Connectors"
