File: kicad/peripherals.kicad_sch (KiCad schematic)
At the start: 9 parts, among them IC1 MAX19777AZA+T, U6 TJA1441BTK/0Z, U7 MC6470

Commit message: Connected all remaining unconnected pins
Parts:
- removed IC1: MAX19777AZA+T, personal:BGA8C35P4X2_143X86X37, symbol personal:MAX19777AZA+T
- added U? (x2): MAX11613EWCT, personal:BGA12N50P3X4_188X221X69N, symbol personal:MAX11613EWCT
Connections:
- net +3V3: now also U?.C1 (VDD), U?.C1 (VDD)
- net GND: now also U7.1 (A5), U?.B1 (GND), U?.B1 (GND), U?.B2 (GND), U?.B2 (GND), U?.B3 (GND), U?.B3 (GND), U?.B4 (GND), U?.B4 (GND), U?.C2 (GND), U?.C2 (GND)
- net GPIO_SCL renamed SCL_1
- net SCL_1: now also U?.C4 (SCL)
- net GPIO_SDA renamed SDA_1
- net SDA_1: now also U?.C3 (SDA)
- new net CONN_19_A8: U?.A1 (AIN0)
- new net CONN_20_A9: U?.A2 (AIN1)
- new net CONN_21_A10: U?.A3 (AIN2)
- new net CONN_22_A11: U?.A4 (AIN3/REF)
- new net SCL_0: U?.C4 (SCL)
- new net SDA_0: U?.C3 (SDA)
Other:
- note added: "NOTE: I2C ADDRESS: 0x34"
- note added: "NOTE: I2C address of accelerometer depends on A5 GND or VDD BIT TYPE ADDRESS 7 bit GND 0x4C 8 bit read GND 0x99 8 bit write GND 0x98 7 bit VCC 0x6C 8 bit read VCC 0xD9 8 bit write VCC 0xD8 MAGNOMETER 0x0C"
- note added: "NOTE: ONLY ON PLUS BOARDS"
- moved on the sheet: R4, TH1

Commit message: Updated schematic with various changes
Increased size of small components
Updated title/spec sheet
Cleaned footprints
Other small changes as well
Parts:
- C32: renamed from C?; footprint (none) -> personal:C_0402_1005Metric
- R6, R7: renamed from R?; footprint (none) -> personal:R_0402_1005Metric
- R8: renamed from R4; footprint personal:R_0201_0603Metric -> personal:R_0402_1005Metric
- gave numbers to parts that had none: 3
- renumbered U6 to U8, U7 to U9
Changed lines of the file:
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@@
   (symbol (lib_id "power:GND") (at 157.48 144.78 0) (unit 1)
     (in_bom yes) (on_board yes) (fields_autoplaced)
-    (property "Reference" "#PWR?" (id 0) (at 157.48 151.13 0)
+    (property "Reference" "#PWR054" (id 0) (at 157.48 151.13 0)
       (effects (font (size 1.27 1.27)) hide)
     )
@@
   (symbol (lib_id "power:+3V3") (at 91.44 111.76 0) (unit 1)
     (in_bom yes) (on_board yes) (fields_autoplaced)
-    (property "Reference" "#PWR?" (id 0) (at 91.44 115.57 0)
+    (property "Reference" "#PWR050" (id 0) (at 91.44 115.57 0)
       (effects (font (size 1.27 1.27)) hide)
     )
@@
   (symbol (lib_id "Device:R_Small") (at 190.5 62.23 0) (unit 1)
     (in_bom yes) (on_board yes) (fields_autoplaced)
-    (property "Reference" "R?" (id 0) (at 193.04 60.9599 0)
+    (property "Reference" "R6" (id 0) (at 193.04 60.9599 0)
       (effects (font (size 1.27 1.27)) (justify left))
     )
@@
       (effects (font (size 1.27 1.27)) (justify left))
     )
-    (property "Footprint" "" (id 2) (at 190.5 62.23 0)
+    (property "Footprint" "personal:R_0402_1005Metric" (id 2) (at 190.5 62.23 0)
       (effects (font (size 1.27 1.27)) hide)
     )
@@
   (symbol (lib_id "power:+3V3") (at 190.5 55.88 0) (unit 1)
     (in_bom yes) (on_board yes) (fields_autoplaced)
-    (property "Reference" "#PWR?" (id 0) (at 190.5 59.69 0)
+    (property "Reference" "#PWR041" (id 0) (at 190.5 59.69 0)
       (effects (font (size 1.27 1.27)) hide)
     )
@@
   (symbol (lib_id "Device:R_Small") (at 204.47 62.23 0) (unit 1)
     (in_bom yes) (on_board yes) (fields_autoplaced)
-    (property "Reference" "R?" (id 0) (at 207.01 60.9599 0)
+    (property "Reference" "R7" (id 0) (at 207.01 60.9599 0)
       (effects (font (size 1.27 1.27)) (justify left))
     )
@@
       (effects (font (size 1.27 1.27)) (justify left))
     )
-    (property "Footprint" "" (id 2) (at 204.47 62.23 0)
+    (property "Footprint" "personal:R_0402_1005Metric" (id 2) (at 204.47 62.23 0)
       (effects (font (size 1.27 1.27)) hide)
     )
@@
   (symbol (lib_id "Device:R_Small") (at 220.98 137.16 0) (unit 1)
     (in_bom yes) (on_board yes)
-    (property "Reference" "R4" (id 0) (at 223.52 135.8899 0)
+    (property "Reference" "R8" (id 0) (at 223.52 135.8899 0)
       (effects (font (size 1.27 1.27)) (justify left))
     )
@@
       (effects (font (size 1.27 1.27)) (justify left))
     )
-    (property "Footprint" "personal:R_0201_0603Metric" (id 2) (at 220.98 137.16 0)
+    (property "Footprint" "personal:R_0402_1005Metric" (id 2) (at 220.98 137.16 0)
       (effects (font (size 1.27 1.27)) hide)
     )
@@
   (symbol (lib_id "personal:MAX11613EWCT") (at 71.12 128.27 0) (unit 1)
     (in_bom yes) (on_board yes) (fields_autoplaced)
-    (property "Reference" "U?" (id 0) (at 71.12 105.41 0))
+    (property "Reference" "U10" (id 0) (at 71.12 105.41 0))
     (property "Value" "MAX11613EWCT" (id 1) (at 71.12 107.95 0))
     (property "Footprint" "personal:BGA12N50P3X4_188X221X69N" (id 2) (at 71.12 128.27 0)
@@
   (symbol (lib_id "power:+3V3") (at 248.92 49.53 0) (unit 1)
     (in_bom yes) (on_board yes) (fields_autoplaced)
-    (property "Reference" "#PWR?" (id 0) (at 248.92 53.34 0)
+    (property "Reference" "#PWR040" (id 0) (at 248.92 53.34 0)
       (effects (font (size 1.27 1.27)) hide)
     )
@@
   (symbol (lib_id "power:+5V") (at 104.14 59.69 0) (unit 1)
     (in_bom yes) (on_board yes) (fields_autoplaced)
-    (property "Reference" "#PWR?" (id 0) (at 104.14 63.5 0)
+    (property "Reference" "#PWR044" (id 0) (at 104.14 63.5 0)
       (effects (font (size 1.27 1.27)) hide)
     )
@@
   (symbol (lib_id "power:GND") (at 162.56 77.47 0) (unit 1)
     (in_bom yes) (on_board yes) (fields_autoplaced)
-    (property "Reference" "#PWR?" (id 0) (at 162.56 83.82 0)
+    (property "Reference" "#PWR047" (id 0) (at 162.56 83.82 0)
       (effects (font (size 1.27 1.27)) hide)
     )
@@
   (symbol (lib_id "Device:C_Small") (at 248.92 54.61 0) (unit 1)
     (in_bom yes) (on_board yes) (fields_autoplaced)
-    (property "Reference" "C?" (id 0) (at 251.46 53.3462 0)
+    (property "Reference" "C32" (id 0) (at 251.46 53.3462 0)
       (effects (font (size 1.27 1.27)) (justify left))
     )
@@
       (effects (font (size 1.27 1.27)) (justify left))
     )
-    (property "Footprint" "" (id 2) (at 248.92 54.61 0)
+    (property "Footprint" "personal:C_0402_1005Metric" (id 2) (at 248.92 54.61 0)
       (effects (font (size 1.27 1.27)) hide)
     )
@@
   (symbol (lib_id "power:GND") (at 92.71 144.78 0) (unit 1)
     (in_bom yes) (on_board yes) (fields_autoplaced)
-    (property "Reference" "#PWR?" (id 0) (at 92.71 151.13 0)
+    (property "Reference" "#PWR053" (id 0) (at 92.71 151.13 0)
       (effects (font (size 1.27 1.27)) hide)
     )
@@
   (symbol (lib_id "power:+3V3") (at 60.96 59.69 0) (unit 1)
     (in_bom yes) (on_board yes) (fields_autoplaced)
-    (property "Reference" "#PWR?" (id 0) (at 60.96 63.5 0)
+    (property "Reference" "#PWR042" (id 0) (at 60.96 63.5 0)
       (effects (font (size 1.27 1.27)) hide)
     )
@@
   (symbol (lib_id "personal:UM3202") (at 67.31 64.77 0) (unit 1)
     (in_bom yes) (on_board yes)
-    (property "Reference" "U?" (id 0) (at 77.47 57.15 0))
+    (property "Reference" "U7" (id 0) (at 77.47 57.15 0))
     (property "Value" "UM3202" (id 1) (at 77.47 59.69 0))
     (property "Footprint" "personal:DFN-8_1.7x1.35mm_P0.4mm" (id 2) (at 76.2 78.74 0)
@@
   (symbol (lib_id "power:+5V") (at 88.9 59.69 0) (unit 1)
     (in_bom yes) (on_board yes) (fields_autoplaced)
-    (property "Reference" "#PWR?" (id 0) (at 88.9 63.5 0)
+    (property "Reference" "#PWR043" (id 0) (at 88.9 63.5 0)
       (effects (font (size 1.27 1.27)) hide)
     )
@@
   (symbol (lib_id "power:+3V3") (at 156.21 111.76 0) (unit 1)
     (in_bom yes) (on_board yes) (fields_autoplaced)
-    (property "Reference" "#PWR?" (id 0) (at 156.21 115.57 0)
+    (property "Reference" "#PWR051" (id 0) (at 156.21 115.57 0)
       (effects (font (size 1.27 1.27)) hide)
     )
@@
   (symbol (lib_id "power:+3.3V") (at 220.98 133.35 0) (unit 1)
     (in_bom yes) (on_board yes)
-    (property "Reference" "#PWR013" (id 0) (at 220.98 137.16 0)
+    (property "Reference" "#PWR052" (id 0) (at 220.98 137.16 0)
       (effects (font (size 1.27 1.27)) hide)
     )
@@
   (symbol (lib_id "power:GND") (at 246.38 88.9 0) (unit 1)
     (in_bom yes) (on_board yes) (fields_autoplaced)
-    (property "Reference" "#PWR?" (id 0) (at 246.38 95.25 0)
+    (property "Reference" "#PWR049" (id 0) (at 246.38 95.25 0)
       (effects (font (size 1.27 1.27)) hide)
     )
@@
   (symbol (lib_id "power:GND") (at 204.47 88.9 0) (unit 1)
     (in_bom yes) (on_board yes) (fields_autoplaced)
-    (property "Reference" "#PWR?" (id 0) (at 204.47 95.25 0)
+    (property "Reference" "#PWR048" (id 0) (at 204.47 95.25 0)
       (effects (font (size 1.27 1.27)) hide)
     )
@@
   (symbol (lib_id "personal:MC6470") (at 226.06 72.39 0) (unit 1)
     (in_bom yes) (on_board yes) (fields_autoplaced)
-    (property "Reference" "U7" (id 0) (at 226.06 52.07 0))
+    (property "Reference" "U9" (id 0) (at 226.06 52.07 0))
     (property "Value" "MC6470" (id 1) (at 213.36 90.17 0)
       (effects (font (size 1.27 1.27)) (justify left bottom))
@@
   (symbol (lib_id "power:GND") (at 220.98 151.765 0) (unit 1)
     (in_bom yes) (on_board yes)
-    (property "Reference" "#PWR014" (id 0) (at 220.98 158.115 0)
+    (property "Reference" "#PWR055" (id 0) (at 220.98 158.115 0)
       (effects (font (size 1.27 1.27)) hide)
     )
@@
   (symbol (lib_id "personal:MAX11613EWCT") (at 135.89 128.27 0) (unit 1)
     (in_bom yes) (on_board yes) (fields_autoplaced)
-    (property "Reference" "U?" (id 0) (at 135.89 105.41 0))
+    (property "Reference" "U11" (id 0) (at 135.89 105.41 0))
     (property "Value" "MAX11613EWCT" (id 1) (at 135.89 107.95 0))
     (property "Footprint" "personal:BGA12N50P3X4_188X221X69N" (id 2) (at 135.89 128.27 0)
@@
   (symbol (lib_id "power:GND") (at 64.77 77.47 0) (unit 1)
     (in_bom yes) (on_board yes) (fields_autoplaced)
-    (property "Reference" "#PWR?" (id 0) (at 64.77 83.82 0)
+    (property "Reference" "#PWR045" (id 0) (at 64.77 83.82 0)
       (effects (font (size 1.27 1.27)) hide)
     )
@@
   (symbol (lib_id "power:GND") (at 101.6 77.47 0) (unit 1)
     (in_bom yes) (on_board yes) (fields_autoplaced)
-    (property "Reference" "#PWR?" (id 0) (at 101.6 83.82 0)
+    (property "Reference" "#PWR046" (id 0) (at 101.6 83.82 0)
       (effects (font (size 1.27 1.27)) hide)
     )
@@
   (symbol (lib_id "personal:TJA1441BTK{slash}0Z") (at 109.22 64.77 0) (unit 1)
     (in_bom yes) (on_board yes)
-    (property "Reference" "U6" (id 0) (at 129.54 53.34 0)
+    (property "Reference" "U8" (id 0) (at 129.54 53.34 0)
       (effects (font (size 1.524 1.524)))
     )
